File: hardware/v0.1a/uPythonFeatherLora.kicad_pcb (KiCad board)
At the start: 2 copper layers, 50.8 x 22.9 mm, 12 parts, among them X1 JSTPH, X3 microUSB

Commit message: Started working on the new design.
Parts:
- removed D+1, D-1: TPB1,27, Adafruit Feather M4 Express:B1,27
- removed X1: JSTPH, Adafruit Feather M4 Express:JSTPH2
- removed X3: microUSB, Adafruit Feather M4 Express:4UCONN_20329_V2
- added J3: USB_OTG, pkl_connectors:Connector_USB_Micro_B_SMD, F.Cu at (124.4, 104.4)
- added J4: Conn_01x02_Male, gkl_conn:S2B-PH-SM4-TB, F.Cu at (133.8, 96.6)
- added U1: ATSAMD51G19A, Housings_DFN_QFN:QFN-48-1EP_7x7mm_Pitch0.5mm, F.Cu at (145.5, 106.1)
- added U2: NCP167, gkl_housings_son:X2SON_4_1.0x1.0mm, F.Cu at (137.1, 110.7)
- added U3: NUP2114, TO_SOT_Packages_SMD:SOT-553, F.Cu at (137.5, 108.4)
- added U4: MCP73832, pkl_housings_sot:SOT-23-5, F.Cu at (134.5, 108.9)
- moved @HOLE0 0.55 mm to (171.3, 95.6)
- moved @HOLE1 0.55 mm to (171.3, 113.3)
- moved U$31 0.55 mm to (125.5, 95.6)
- moved U$32 0.55 mm to (125.5, 113.3)
- moved CHG1 0.55 mm to (125.4, 110.3)
- moved JP1 0.55 mm to (148.4, 114.6)
- moved JP3 0.55 mm to (153.5, 94.3)
- moved L1 0.55 mm to (125.6, 98.5)
Other:
- outline, holes or cut-outs redrawn
